File: robo1.kicad_pcb (KiCad board)
At the start: 2 copper layers, 122.2 x 76.9 mm, 36 parts, among them J1 Conn_02x05_Odd_Even, J2 Conn_02x05_Odd_Even, J3 Conn_01x04_Pin, J4 Conn_01x04_Pin, J5 Screw_Terminal_01x02, J6 Screw_Terminal_01x02, J7 Conn_01x03_Pin, J8 Conn_01x03_Pin, SW1 SW_Push, SW2 SW_Push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

Commit message: update to use ad5590 and pb encoder
Parts:
- added SW4: RotaryEncoder_Switch, Rotary_Encoder:RotaryEncoder_Alps_EC11E-Switch_Vertical_H20mm_CircularMountingHoles, F.Cu at (151.2, 95.5)
- added SW5: Menu, Button_Switch_THT:SW_PUSH_6mm, F.Cu at (127.1, 114.1)
- added U2: AD5593R, Package_SO:TSSOP-16_4.4x5mm_P0.65mm, F.Cu at (96.8, 111.3)
- SW1: value SW_Push -> ESTOP
- SW2: value SW_Push -> Right
- SW3: value SW_Push -> Left
- moved SW2 54.9 mm to (104.2, 113.8)
- moved D4 48.4 mm to (150.1, 58.9)
- moved SW1 40.7 mm to (146.9, 48.8)
- moved SW3 15.8 mm to (150.9, 114.1)
- moved REF** 9.92 mm to (118.4, 108.5)
- moved REF** 8.93 mm to (119.6, 85.3)
- moved Brd1 7.69 mm to (130.7, 97.6)
- moved R9 7.68 mm to (107.4, 95.2)
- moved REF** 7.33 mm to (141.5, 85.9)
- moved REF** 6.86 mm to (141.7, 108.2)
- moved R8 6.72 mm to (105.7, 90.2)
- moved D1 6.57 mm to (111.8, 102.9)
- moved D2 6.57 mm to (111.8, 100.3)
- moved R6 5.59 mm to (106.6, 102.9)
- moved D3 2.41 mm to (113.9, 80.3)
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Connections:
- R8 pad 1: Net-(U1-GPIO18) -> Net-(U1-GPIO20)
- SW1 pad 2: /BTN_UP -> unconnected-(SW1-Pad2)
- U1 pad 24: Net-(U1-GPIO18) -> /I2C1_SDA
- U1 pad 26: /I2C1_SDA -> Net-(U1-GPIO20)
Routing:
- net Net-(U1-GPIO16): track 11.4 -> 0.00 mm
- net Net-(U1-GPIO18): track 9.32 -> 0.00 mm
- net Net-(D2-A): track 8.08 -> 0.00 mm
- net Net-(U1-GPIO17): track 7.62 -> 0.00 mm
- net GND: track 6.53 -> 0.00 mm, vias 3 -> 0
- net Net-(D4-A): track 6.16 -> 0.00 mm
- net /I2C1_SDA: track 0.00 -> 5.59 mm
- net Net-(D1-A): track 4.27 -> 0.00 mm
